Commit message: Fix namespaced wheels

File: irobot_create_common/irobot_create_description/urdf/create3.urdf.xacro (robot description, xacro)
@@ -94,10 +94,10 @@
   </xacro:bumper>
   <!-- Wheels with mechanical wheel drop -->
-  <!-- <xacro:wheel_with_wheeldrop name="left" gazebo="$(arg gazebo)" namespace="$(arg namespace)">
+  <xacro:wheel_with_wheeldrop name="left" gazebo="$(arg gazebo)" namespace="$(arg namespace)">
     <origin xyz="0 ${distance_between_wheels/2} ${wheel_drop_z  + base_link_z_offset}" rpy="${-pi/2} 0 0"/>
   </xacro:wheel_with_wheeldrop>
   <xacro:wheel_with_wheeldrop name="right" gazebo="$(arg gazebo)" namespace="$(arg namespace)">
     <origin xyz="0 ${-distance_between_wheels/2} ${wheel_drop_z  + base_link_z_offset}" rpy="${-pi/2} 0 0"/>
-  </xacro:wheel_with_wheeldrop> -->
+  </xacro:wheel_with_wheeldrop>
   <!-- Caster wheel -->
   <xacro:caster name="front_caster" parent_link="base_link">

File: irobot_create_common/irobot_create_description/urdf/wheel.urdf.xacro (robot description, xacro)
@@ -5,13 +5,13 @@
   <xacro:property name="radius" value="${3.575*cm2m}" />
   <xacro:property name="width"  value="${1.5*cm2m}" />
-  <xacro:property name="wheel_link_name"  value="${ns_prefix}${name}_wheel"/>
+  <xacro:property name="wheel_link_name"  value="${name}_wheel"/>
   <xacro:property name="wheel_joint_name" value="${wheel_link_name}_joint"/>
-  <joint name="${wheel_joint_name}" type="continuous">
+  <joint name="${ns_prefix}${wheel_joint_name}" type="continuous">
     <parent link="${ns_prefix}${parent_link}"/>
-    <child link="${wheel_link_name}"/>
+    <child link="${ns_prefix}${wheel_link_name}"/>
     <xacro:insert_block name="origin"/>
     <axis xyz="0 0 1"/>
   </joint>
-  <link name="${wheel_link_name}">
+  <link name="${ns_prefix}${wheel_link_name}">
     <visual>
       <geometry>
@@ -29,5 +29,5 @@
       length="${width}" />
   </link>
-  <gazebo reference="${wheel_link_name}">
+  <gazebo reference="${ns_prefix}${wheel_link_name}">
     <mu1>1.0</mu1>
     <mu2>1.0</mu2>
@@ -43,5 +43,5 @@
         <plugin>gazebo_ros2_control/GazeboSystem</plugin>
       </hardware>
-      <joint name="${wheel_joint_name}">
+      <joint name="${ns_prefix}${wheel_joint_name}">
         <state_interface name="velocity" />
         <state_interface name="position" />
@@ -55,5 +55,5 @@
         <plugin>ign_ros2_control/IgnitionSystem</plugin>
       </hardware>
-      <joint name="${wheel_joint_name}">
+      <joint name="${ns_prefix}${wheel_joint_name}">
         <state_interface name="velocity" />
         <state_interface name="position" />

File: irobot_create_common/irobot_create_description/urdf/wheel_drop.urdf.xacro (robot description, xacro)
@@ -17,9 +17,9 @@
   <xacro:property name="wd_mass" value="0.05"/>
   <xacro:property name="update_rate"   value="62" />
-  <xacro:property name="wd_link_name"  value="$wheel_drop_${name}"/>
+  <xacro:property name="wd_link_name"  value="wheel_drop_${name}"/>
   <xacro:property name="wd_joint_name" value="${wd_link_name}_joint"/>
-  <joint name="{ns_prefix}${wd_joint_name}" type="prismatic">
+  <joint name="${ns_prefix}${wd_joint_name}" type="prismatic">
     <parent link="${ns_prefix}${parent_link}"/>
-    <child link="{ns_prefix}${wd_link_name}"/>
+    <child link="${ns_prefix}${wd_link_name}"/>
     <xacro:insert_block name="origin"/>
     <axis xyz="0 1 0"/>
@@ -29,5 +29,5 @@
   </joint>
   <!-- Gazebo parameters to simulate a spring -->
-  <gazebo reference="{ns_prefix}${wd_joint_name}">
+  <gazebo reference="${ns_prefix}${wd_joint_name}">
     <provideFeedback>false</provideFeedback>
     <implicitSpringDamper>true</implicitSpringDamper>
@@ -37,5 +37,5 @@
     <springReference>${detection_threshold}</springReference>
   </gazebo>
-  <link name="{ns_prefix}${wd_link_name}">
+  <link name="${ns_prefix}${wd_link_name}">
     <xacro:inertial_cuboid mass="${wd_mass}" x="${wd_size}" y="${wd_size}" z="${wd_size}"/>
   </link>
@@ -49,6 +49,6 @@
         <update_rate>${update_rate}</update_rate>
         <detection_threshold>${detection_threshold}</detection_threshold>
-        <joint_name>{ns_prefix}${wd_joint_name}</joint_name>
-        <frame_id>{ns_prefix}${wd_link_name}</frame_id>
+        <joint_name>${ns_prefix}${wd_joint_name}</joint_name>
+        <frame_id>${ns_prefix}${wd_link_name}</frame_id>
       </plugin>
     </gazebo>
